Commit message: Added four wheeled robot

File: description/camera.xacro (robot description, xacro)
@@ -5,5 +5,5 @@
         <parent link="chassis"/>
         <child link="camera_link"/>
-        <origin xyz="0.35 0 0.08" rpy="0 0 0"/>
+        <origin xyz="0.175 0 0.08" rpy="0 0 0"/>
     </joint>
     <link name="camera_link">
@@ -12,5 +12,5 @@
                 <box size="0.010 0.03 0.03"/>
             </geometry>
-            <material name="blue"/>
+            <material name="orange"/>
         </visual>
     </link>
@@ -24,5 +24,5 @@
     <!-- Camera Gazebo Sensor Plugin -->
     <gazebo reference="camera_link">
-        <material>Gazebo/Blue</material>
+        <material>Gazebo/Orange</material>
         <sensor name="camera" type="camera">
             <pose> 0 0 0 0 0 0 </pose>

File: description/depth_camera.xacro (robot description, xacro)
@@ -5,5 +5,5 @@
         <parent link="chassis"/>
         <child link="camera_link"/>
-        <origin xyz="0.35 0 0.08" rpy="0 0 0"/>
+        <origin xyz="0.175 0 0.05" rpy="0 0 0"/>
     </joint>
     <link name="camera_link">
@@ -12,5 +12,5 @@
                 <box size="0.010 0.03 0.03"/>
             </geometry>
-            <material name="red"/>
+            <material name="purple"/>
         </visual>
     </link>
@@ -24,5 +24,5 @@
     <!-- Deepth Camera Gazebo Sensor Plugin -->
     <gazebo reference="camera_link">
-        <material>Gazebo/Red</material>
+        <material>Gazebo/Purple</material>
         <sensor name="camera" type="depth">
             <pose> 0 0 0 0 0 0 </pose>

File: description/diff_bot.urdf.xacro (robot description, xacro)
@@ -5,5 +5,5 @@
     <xacro:include filename="inertials.xacro"/>
     <xacro:include filename="materials.xacro"/>
-    <!-- Include sensors (currently only lidar, camera and deepth camera supported) -->
+    <!-- Include sensors (currently only lidar, camera and depth camera supported) -->
     <xacro:include filename="lidar.xacro"/>
     <!-- <xacro:include filename="camera.xacro"/> -->
@@ -18,9 +18,9 @@
     <xacro:property name="wheel_mass" value="0.3"/>
     <xacro:property name="wheel_offset_x" value="0.13"/>
-    <xacro:property name="wheel_offset_y" value="0.169"/>
+    <xacro:property name="wheel_offset_y" value="${chassis_width/2 + wheel_thickness/2}"/>
     <xacro:property name="wheel_offset_z" value="0.0"/>
     <xacro:property name="caster_wheel_radius" value="0.032225"/>
     <xacro:property name="caster_wheel_mass" value="0.2"/>
-    <xacro:property name="caster_wheel_offset_x" value="${chassis_length + 0.0}"/>
+    <xacro:property name="caster_wheel_offset_x" value="${chassis_length/2}"/>
     <xacro:property name="caster_wheel_offset_z" value="${wheel_offset_z - wheel_radius + caster_wheel_radius}"/>
     <!-- Base Link -->
@@ -37,9 +37,9 @@
         <parent link="base_link"/>
         <child link="chassis"/>
-        <origin xyz="${-wheel_offset_x} 0 ${-wheel_offset_z}"/>
+        <origin xyz="0 0 0"/>
     </joint>
     <link name="chassis">
         <visual>
-            <origin xyz="${chassis_length/2} 0 ${chassis_height/2}"/>
+            <origin xyz="0 0 ${chassis_height/2}"/>
             <geometry>
                 <box size="${chassis_length} ${chassis_width} ${chassis_height}"/>
@@ -48,5 +48,5 @@
         </visual>
         <collision>
-            <origin xyz="${chassis_length/2} 0 ${chassis_height/2}"/>
+            <origin xyz="0 0 ${chassis_height/2}"/>
             <geometry>
                 <box size="${chassis_length} ${chassis_width} ${chassis_height}"/>
@@ -54,5 +54,5 @@
         </collision>
         <xacro:inertial_box mass="0.5" x="${chassis_length}" y="${chassis_width}" z="${chassis_height}">
-            <origin xyz="${chassis_length/2} 0 ${chassis_height/2}" rpy="0 0 0"/>
+            <origin xyz="0 0 ${chassis_height/2}" rpy="0 0 0"/>
         </xacro:inertial_box>
     </link>
@@ -61,5 +61,5 @@
         <parent link="base_link"/>
         <child link="left_wheel"/>
-        <origin xyz="0 ${wheel_offset_y} 0" rpy="-${pi/2} 0 0" />
+        <origin xyz="${-wheel_offset_x} ${wheel_offset_y} 0" rpy="-${pi/2} 0 0" />
         <axis xyz="0 0 1"/>
     </joint>
@@ -84,5 +84,5 @@
         <parent link="base_link"/>
         <child link="right_wheel"/>
-        <origin xyz="0 ${-wheel_offset_y} 0" rpy="${pi/2} 0 0" />
+        <origin xyz="${-wheel_offset_x} ${-wheel_offset_y} 0" rpy="${pi/2} 0 0" />
         <axis xyz="0 0 -1"/>
     </joint>

File: description/lidar.xacro (robot description, xacro)
@@ -5,5 +5,5 @@
         <parent link="chassis"/>
         <child link="laser_frame"/>
-        <origin xyz="0.122 0 0.09" rpy="0 0 0"/>
+        <origin xyz="0 0 0.1" rpy="0 0 0"/>
     </joint>
     <link name="laser_frame">

Commit message: Upgraded to Gazebo Fortress

File: description/camera.xacro (robot description, xacro)
@@ -27,7 +27,11 @@
         <sensor name="camera" type="camera">
             <pose> 0 0 0 0 0 0 </pose>
+            <always_on>true</always_on>
             <visualize>true</visualize>
-            <update_rate>10</update_rate>
+            <update_rate>30</update_rate>
+            <topic>camera/image_raw</topic>
+            <gz_frame_id>camera_link_optical</gz_frame_id>
             <camera>
+                <camera_info_topic>camera/camera_info</camera_info_topic>
                 <horizontal_fov>1.089</horizontal_fov>
                 <image>
@@ -41,7 +45,4 @@
                 </clip>
             </camera>
-            <plugin name="camera_controller" filename="libgazebo_ros_camera.so">
-                <frame_name>camera_link_optical</frame_name>
-            </plugin>
         </sensor>
     </gazebo>

File: description/common.xacro (robot description, xacro)
@@ -1,5 +1,6 @@
 <?xml version="1.0"?>
 <robot xmlns:xacro="http://www.ros.org/wiki/xacro" >
-    <!-- This file contains the inertial macros used across the URDF files -->
+    <!-- This file contains the macros used across the URDF files -->
+    <!-- Inertial Macros -->
     <!-- Inertial Sphere Macros -->
     <xacro:macro name="inertial_sphere" params="mass radius *origin">
@@ -32,4 +33,28 @@
         </inertial>
     </xacro:macro>
-    <!-- Add more here -->
+    <!-- Material Macros -->
+    <material name="white">
+        <color rgba="1 1 1 1" />
+    </material>
+    <material name="orange">
+        <color rgba="1 0.3 0.1 1"/>
+    </material>
+    <material name="blue">
+        <color rgba="0.2 0.2 1 1"/>
+    </material>
+    <material name="black">
+        <color rgba="0 0 0 1"/>
+    </material>
+    <material name="red">
+        <color rgba="1 0 0 1"/>
+    </material>
+    <material name="grey">
+        <color rgba="0.631 0.631 0.631 1"/>
+    </material>
+    <material name="purple">
+        <color rgba="0.78 0.153 0.71 1"/>
+    </material>
+    <material name="green">
+        <color rgba="0.149 0.612 0.082 1"/>
+    </material>
 </robot>

File: description/diff_bot.urdf.xacro (robot description, xacro)
@@ -2,12 +2,11 @@
 <robot xmlns:xacro="http://www.ros.org/wiki/xacro"  name="robot">
     <!-- Main URDF file for Differential Drive Robot -->
-    <!-- Include general xacro files -->
-    <xacro:include filename="inertials.xacro"/>
-    <xacro:include filename="materials.xacro"/>
+    <!-- Include general xacro macros -->
+    <xacro:include filename="common.xacro"/>
     <!-- Include sensors -->
     <xacro:include filename="lidar.xacro"/>
-    <xacro:include filename="depth_camera.xacro"/>
-    <!-- <xacro:include filename="camera.xacro"/> -->
+    <xacro:include filename="camera.xacro"/>
     <!-- <xacro:include filename="3dlidar.xacro"/> -->
+    <!-- <xacro:include filename="depth_camera.xacro"/> -->
     <!-- Robot Variables -->
     <xacro:property name="chassis_length" value="0.35"/>
@@ -141,22 +140,30 @@
         <mu2 value="0.001"/>
     </gazebo>
-    <!-- Gazebo plugin for differential drive robots -->
+    <!-- Gazebo plugins -->
     <gazebo>
-        <plugin name="diff_drive" filename="libgazebo_ros_diff_drive.so">
-            <!-- Wheel Information -->
+        <!-- Differential Drive Robot -->
+        <plugin filename="gz-sim-diff-drive-system" name="gz::sim::systems::DiffDrive">
+            <!-- Wheels -->
             <left_joint>left_wheel_joint</left_joint>
             <right_joint>right_wheel_joint</right_joint>
             <wheel_separation>${wheel_offset_y*2}</wheel_separation>
-            <wheel_diameter>${wheel_radius*2}</wheel_diameter>
+            <wheel_radius>${wheel_radius}</wheel_radius>
             <!-- Limits -->
-            <max_wheel_torque>80</max_wheel_torque>
-            <max_wheel_acceleration>6.0</max_wheel_acceleration>
+            <max_linear_acceleration>6.0</max_linear_acceleration>
             <!-- Frames -->
-            <odometry_frame>odom</odometry_frame>
-            <robot_base_frame>base_link</robot_base_frame>
+            <frame_id>odom</frame_id>
+            <child_frame_id>base_link</child_frame_id>
             <!-- Output -->
-            <publish_odom>true</publish_odom>
-            <publish_odom_tf>true</publish_odom_tf>
-            <publish_wheel_tf>true</publish_wheel_tf>
+            <tf_topic>/tf</tf_topic>
+            <topic>cmd_vel</topic>
+            <odom_topic>odom</odom_topic>
+            <odom_publisher_frequency>30</odom_publisher_frequency>
+        </plugin>
+        <!-- Joint State Publisher -->
+        <plugin filename="gz-sim-joint-state-publisher-system"
+            name="gz::sim::systems::JointStatePublisher">
+            <topic>joint_states</topic>
+            <joint_name>left_wheel_joint</joint_name>
+            <joint_name>right_wheel_joint</joint_name>
         </plugin>
     </gazebo>

File: description/lidar.xacro (robot description, xacro)
@@ -23,12 +23,15 @@
         </xacro:inertial_cylinder>
     </link>
-    <!-- 2D Lidar Gazebo Sensor Plugin  -->
+    <!-- 2D Lidar New Gazebo Sensor Plugin  -->
     <gazebo reference="laser_frame">
         <material>Gazebo/Black</material>
-        <sensor name="laser" type="ray">
+        <sensor name="laser" type="gpu_lidar">
             <pose> 0 0 0 0 0 0 </pose>
+            <always_on>true</always_on>
             <visualize>true</visualize>
             <update_rate>10</update_rate>
-            <ray>
+            <topic>scan</topic>
+            <gz_frame_id>laser_frame</gz_frame_id>
+            <lidar>
                 <scan>
                     <horizontal>
@@ -42,12 +45,5 @@
                     <max>12</max>
                 </range>
-            </ray>
-            <plugin name="laser_controller" filename="libgazebo_ros_ray_sensor.so">
-                <ros>
-                    <argument>~/out:=scan</argument>
-                </ros>
-                <output_type>sensor_msgs/LaserScan</output_type>
-                <frame_name>laser_frame</frame_name>
-            </plugin>
+            </lidar>
         </sensor>
     </gazebo>
