Commit message: Added depth camera to sim

File: description/depth_camera.xacro (robot description, xacro)
@@ -1,5 +1,5 @@
 <?xml version="1.0"?>
 <robot xmlns:xacro="http://www.ros.org/wiki/xacro" >
-    <!-- Camera's urdf -->
+    <!-- Depth camera's urdf -->
     <joint name="camera_joint" type="fixed">
         <parent link="chassis"/>
@@ -15,5 +15,5 @@
         </visual>
     </link>
-    <!-- Camera Optical link -->
+    <!-- Depth camera Optical link -->
     <joint name="camera_optical_joint" type="fixed">
         <parent link="camera_link"/>
@@ -22,15 +22,16 @@
     </joint>
     <link name="camera_link_optical"></link>
-    <!-- Camera Gazebo Sensor Plugin -->
+    <!-- Depth camera Gazebo Sensor Plugin -->
     <gazebo reference="camera_link">
         <material>Gazebo/Black</material>
-        <sensor name="camera" type="camera">
+        <sensor name="rgbd_camera" type="rgbd_camera">
             <pose> 0 0 0 0 0 0 </pose>
             <always_on>true</always_on>
             <visualize>true</visualize>
             <update_rate>30</update_rate>
-            <topic>camera/image</topic>
-            <gz_frame_id>camera_link_optical</gz_frame_id>
+            <topic>camera</topic>
+            <gz_frame_id>camera_link</gz_frame_id>
             <camera>
+                <optical_frame_id>camera_link_optical</optical_frame_id>
                 <camera_info_topic>camera/camera_info</camera_info_topic>
                 <horizontal_fov>1.089</horizontal_fov>

File: description/diff_bot.urdf.xacro (robot description, xacro)
@@ -1,4 +1,4 @@
 <?xml version="1.0"?>
-<robot xmlns:xacro="http://www.ros.org/wiki/xacro"  name="robot">
+<robot xmlns:xacro="http://www.ros.org/wiki/xacro"  name="diff_bot">
     <!-- Main URDF file for Differential Drive Robot -->
     <!-- Include general xacro macros -->
@@ -6,7 +6,7 @@
     <!-- Include sensors -->
     <xacro:include filename="lidar.xacro"/>
-    <xacro:include filename="camera.xacro"/>
+    <xacro:include filename="depth_camera.xacro"/>
+    <!-- <xacro:include filename="camera.xacro"/> -->
     <!-- <xacro:include filename="3dlidar.xacro"/> -->
-    <!-- <xacro:include filename="depth_camera.xacro"/> -->
     <!-- Robot Variables -->
     <xacro:property name="chassis_length" value="0.35"/>
@@ -114,5 +114,5 @@
                 <sphere radius="${caster_wheel_radius}"/>
             </geometry>
-            <material name="white"/>
+            <material name="black"/>
         </visual>
         <collision>
@@ -136,5 +136,5 @@
     </gazebo>
     <gazebo reference="caster_wheel">
-        <material>Gazebo/White</material>
+        <material>Gazebo/Black</material>
         <mu1 value="0.001"/>
         <mu2 value="0.001"/>
@@ -161,6 +161,5 @@
         </plugin>
         <!-- Joint State Publisher -->
-        <plugin filename="gz-sim-joint-state-publisher-system"
-            name="gz::sim::systems::JointStatePublisher">
+        <plugin filename="gz-sim-joint-state-publisher-system" name="gz::sim::systems::JointStatePublisher">
             <topic>joint_states</topic>
             <joint_name>left_wheel_joint</joint_name>

File: description/lidar.xacro (robot description, xacro)
@@ -12,5 +12,5 @@
                 <cylinder radius="0.05" length="0.05"/>
             </geometry>
-            <material name="black"/>
+            <material name="grey"/>
         </visual>
         <collision>
@@ -25,5 +25,5 @@
     <!-- 2D Lidar New Gazebo Sensor Plugin  -->
     <gazebo reference="laser_frame">
-        <material>Gazebo/Black</material>
+        <material>Gazebo/Grey</material>
         <sensor name="laser" type="gpu_lidar">
             <pose> 0 0 0 0 0 0 </pose>
