Commit message: Added camera to simulation

File: description/diff_bot.urdf.xacro (robot description, xacro)
@@ -5,20 +5,21 @@
     <xacro:include filename="inertials.xacro"/>
     <xacro:include filename="materials.xacro"/>
-    <!-- Include sensors (currently only lidar supported) -->
+    <!-- Include sensors (currently only lidar and camera supported) -->
     <xacro:include filename="lidar.xacro"/>
+    <xacro:include filename="camera.xacro"/>
     <!-- Robot Variables -->
-    <xacro:property name="chassis_length" value="0.448"/>
+    <xacro:property name="chassis_length" value="0.35"/>
     <xacro:property name="chassis_width" value="0.3"/>
-    <xacro:property name="chassis_height" value="0.07913"/>
-    <xacro:property name="chassis_mass" value="6.0"/>
-    <xacro:property name="wheel_radius" value="0.0775"/>
-    <xacro:property name="wheel_thickness" value="0.03886"/>
-    <xacro:property name="wheel_mass" value="0.5"/>
-    <xacro:property name="wheel_offset_x" value="0.07388"/>
+    <xacro:property name="chassis_height" value="0.08"/>
+    <xacro:property name="chassis_mass" value="4.0"/>
+    <xacro:property name="wheel_radius" value="0.05"/>
+    <xacro:property name="wheel_thickness" value="0.018"/>
+    <xacro:property name="wheel_mass" value="0.3"/>
+    <xacro:property name="wheel_offset_x" value="0.13"/>
     <xacro:property name="wheel_offset_y" value="0.169"/>
     <xacro:property name="wheel_offset_z" value="0.0"/>
     <xacro:property name="caster_wheel_radius" value="0.032225"/>
     <xacro:property name="caster_wheel_mass" value="0.2"/>
-    <xacro:property name="caster_wheel_offset_x" value="0.45862"/>
+    <xacro:property name="caster_wheel_offset_x" value="${chassis_length + 0.0}"/>
     <xacro:property name="caster_wheel_offset_z" value="${wheel_offset_z - wheel_radius + caster_wheel_radius}"/>
     <!-- Base Link -->
@@ -147,6 +148,6 @@
             <wheel_diameter>${wheel_radius*2}</wheel_diameter>
             <!-- Limits -->
-            <max_wheel_torque>200</max_wheel_torque>
-            <max_wheel_acceleration>10.0</max_wheel_acceleration>
+            <max_wheel_torque>80</max_wheel_torque>
+            <max_wheel_acceleration>6.0</max_wheel_acceleration>
             <!-- Frames -->
             <odometry_frame>odom</odometry_frame>

Commit message: Added 3D lidar to sim

File: description/diff_bot.urdf.xacro (robot description, xacro)
@@ -7,4 +7,5 @@
     <xacro:include filename="lidar.xacro"/>
     <xacro:include filename="depth_camera.xacro"/>
+    <!-- Extra sensors -->
     <!-- <xacro:include filename="camera.xacro"/> -->
     <!-- <xacro:include filename="3dlidar.xacro"/> -->
@@ -17,5 +18,5 @@
     <xacro:property name="wheel_thickness" value="0.018"/>
     <xacro:property name="wheel_mass" value="0.3"/>
-    <xacro:property name="wheel_offset_x" value="0.13"/>
+    <xacro:property name="wheel_offset_x" value="0.1"/>
     <xacro:property name="wheel_offset_y" value="${chassis_width/2 + wheel_thickness/2}"/>
     <xacro:property name="wheel_offset_z" value="0.0"/>
