Commit message: Added four wheel robot

File: description/four_wheel.urdf.xacro (robot description, xacro)
@@ -1,6 +1,6 @@
 <?xml version="1.0"?>
-<robot xmlns:xacro="http://www.ros.org/wiki/xacro"  name="diff_bot">
-    <!-- Main URDF file for Two Wheeled Differential Drive Robot -->
-    <!-- Include general xacro macros -->
+<robot xmlns:xacro="http://www.ros.org/wiki/xacro"  name="four_wheel_diff_bot">
+    <!-- Main URDF file for Four Wheeled Differential Drive Robot -->
+    <!-- Include general xacro files -->
     <xacro:include filename="common.xacro"/>
     <!-- Include sensors -->
@@ -18,11 +18,7 @@
     <xacro:property name="wheel_thickness" value="0.018"/>
     <xacro:property name="wheel_mass" value="0.3"/>
-    <xacro:property name="wheel_offset_x" value="0.1"/>
+    <xacro:property name="wheel_offset_x" value="0.13"/>
     <xacro:property name="wheel_offset_y" value="${chassis_width/2 + wheel_thickness/2}"/>
     <xacro:property name="wheel_offset_z" value="0.0"/>
-    <xacro:property name="caster_wheel_radius" value="0.032225"/>
-    <xacro:property name="caster_wheel_mass" value="0.2"/>
-    <xacro:property name="caster_wheel_offset_x" value="${chassis_length/2}"/>
-    <xacro:property name="caster_wheel_offset_z" value="${wheel_offset_z - wheel_radius + caster_wheel_radius}"/>
     <!-- Base Link -->
     <link name="base_link"></link>
@@ -46,5 +42,5 @@
                 <box size="${chassis_length} ${chassis_width} ${chassis_height}"/>
             </geometry>
-            <material name="red"/>
+            <material name="blue"/>
         </visual>
         <collision>
@@ -58,17 +54,17 @@
         </xacro:inertial_box>
     </link>
-    <!-- Left Wheel -->
-    <joint name="left_wheel_joint" type="continuous">
+    <!-- Front Left Wheel -->
+    <joint name="front_left_wheel_joint" type="continuous">
         <parent link="base_link"/>
-        <child link="left_wheel"/>
-        <origin xyz="${-wheel_offset_x} ${wheel_offset_y} 0" rpy="-${pi/2} 0 0" />
+        <child link="front_left_wheel"/>
+        <origin xyz="${wheel_offset_x} ${wheel_offset_y} 0" rpy="-${pi/2} 0 0" />
         <axis xyz="0 0 1"/>
     </joint>
-    <link name="left_wheel">
+    <link name="front_left_wheel">
         <visual>
             <geometry>
                 <cylinder radius="${wheel_radius}" length="${wheel_thickness}"/>
             </geometry>
-            <material name="black"/>
+            <material name="white"/>
         </visual>
         <collision>
@@ -81,17 +77,17 @@
         </xacro:inertial_cylinder>
     </link>
-    <!-- Right Wheel -->
-    <joint name="right_wheel_joint" type="continuous">
+    <!-- Front Right Wheel -->
+    <joint name="front_right_wheel_joint" type="continuous">
         <parent link="base_link"/>
-        <child link="right_wheel"/>
-        <origin xyz="${-wheel_offset_x} ${-wheel_offset_y} 0" rpy="${pi/2} 0 0" />
+        <child link="front_right_wheel"/>
+        <origin xyz="${wheel_offset_x} ${-wheel_offset_y} 0" rpy="${pi/2} 0 0" />
         <axis xyz="0 0 -1"/>
     </joint>
-    <link name="right_wheel">
+    <link name="front_right_wheel">
         <visual>
             <geometry>
                 <cylinder radius="${wheel_radius}" length="${wheel_thickness}"/>
             </geometry>
-            <material name="black"/>
+            <material name="white"/>
         </visual>
         <collision>
@@ -104,52 +100,81 @@
         </xacro:inertial_cylinder>
     </link>
-    <!-- Caster Wheel -->
-    <joint name="caster_wheel_joint" type="fixed">
-        <parent link="chassis"/>
-        <child link="caster_wheel"/>
-        <origin xyz="${caster_wheel_offset_x} 0 ${caster_wheel_offset_z}"/>
+    <!-- Rear Left Wheel -->
+    <joint name="rear_left_wheel_joint" type="continuous">
+        <parent link="base_link"/>
+        <child link="rear_left_wheel"/>
+        <origin xyz="${-wheel_offset_x} ${wheel_offset_y} 0" rpy="-${pi/2} 0 0" />
+        <axis xyz="0 0 1"/>
     </joint>
-    <link name="caster_wheel">
+    <link name="rear_left_wheel">
         <visual>
             <geometry>
-                <sphere radius="${caster_wheel_radius}"/>
+                <cylinder radius="${wheel_radius}" length="${wheel_thickness}"/>
             </geometry>
-            <material name="black"/>
+            <material name="white"/>
         </visual>
         <collision>
             <geometry>
-                <sphere radius="${caster_wheel_radius}"/>
+                <sphere radius="${wheel_radius}"/>
             </geometry>
         </collision>
-        <xacro:inertial_sphere mass="${caster_wheel_mass}" radius="${caster_wheel_radius}">
+        <xacro:inertial_cylinder mass="${wheel_mass}" length="${wheel_thickness}" radius="${wheel_radius}">
             <origin xyz="0 0 0" rpy="0 0 0"/>
-        </xacro:inertial_sphere>
+        </xacro:inertial_cylinder>
+    </link>
+    <!-- Rear Right Wheel -->
+    <joint name="rear_right_wheel_joint" type="continuous">
+        <parent link="base_link"/>
+        <child link="rear_right_wheel"/>
+        <origin xyz="${-wheel_offset_x} ${-wheel_offset_y} 0" rpy="${pi/2} 0 0" />
+        <axis xyz="0 0 -1"/>
+    </joint>
+    <link name="rear_right_wheel">
+        <visual>
+            <geometry>
+                <cylinder radius="${wheel_radius}" length="${wheel_thickness}"/>
+            </geometry>
+            <material name="white"/>
+        </visual>
+        <collision>
+            <geometry>
+                <sphere radius="${wheel_radius}"/>
+            </geometry>
+        </collision>
+        <xacro:inertial_cylinder mass="${wheel_mass}" length="${wheel_thickness}" radius="${wheel_radius}">
+            <origin xyz="0 0 0" rpy="0 0 0"/>
+        </xacro:inertial_cylinder>
     </link>
     <!-- Gazebo -->
     <gazebo reference="chassis">
-        <material>Gazebo/Red</material>
+        <material>Gazebo/Blue</material>
     </gazebo>
-    <gazebo reference="left_wheel">
-        <material>Gazebo/Black</material>
+    <gazebo reference="front_left_wheel">
+        <material>Gazebo/White</material>
     </gazebo>
-    <gazebo reference="right_wheel">
-        <material>Gazebo/Black</material>
+    <gazebo reference="front_right_wheel">
+        <material>Gazebo/White</material>
     </gazebo>
-    <gazebo reference="caster_wheel">
-        <material>Gazebo/Black</material>
-        <mu1 value="0.001"/>
-        <mu2 value="0.001"/>
+    <gazebo reference="rear_left_wheel">
+        <material>Gazebo/White</material>
     </gazebo>
-    <!-- Gazebo plugins -->
+    <gazebo reference="rear_right_wheel">
+        <material>Gazebo/White</material>
+    </gazebo>
     <gazebo>
-        <!-- Differential Drive Robot -->
+        <!-- Four Wheeled Differential Drive Robot -->
         <plugin filename="gz-sim-diff-drive-system" name="gz::sim::systems::DiffDrive">
             <!-- Wheels -->
-            <left_joint>left_wheel_joint</left_joint>
-            <right_joint>right_wheel_joint</right_joint>
+            <left_joint>rear_left_wheel_joint</left_joint>
+            <left_joint>front_left_wheel_joint</left_joint>
+            <right_joint>rear_right_wheel_joint</right_joint>
+            <right_joint>front_right_wheel_joint</right_joint>
+            <!-- Wheel params -->
+            <wheel_radius>${wheel_radius}</wheel_radius>
             <wheel_separation>${wheel_offset_y*2}</wheel_separation>
             <wheel_radius>${wheel_radius}</wheel_radius>
+            <wheel_separation>${wheel_offset_y*2}</wheel_separation>
             <!-- Limits -->
-            <max_linear_acceleration>6.0</max_linear_acceleration>
+            <max_linear_acceleration>2.0</max_linear_acceleration>
             <!-- Frames -->
             <frame_id>odom</frame_id>
@@ -164,6 +189,8 @@
         <plugin filename="gz-sim-joint-state-publisher-system" name="gz::sim::systems::JointStatePublisher">
             <topic>joint_states</topic>
-            <joint_name>left_wheel_joint</joint_name>
-            <joint_name>right_wheel_joint</joint_name>
+            <joint_name>front_left_wheel_joint</joint_name>
+            <joint_name>front_right_wheel_joint</joint_name>
+            <joint_name>rear_left_wheel_joint</joint_name>
+            <joint_name>rear_right_wheel_joint</joint_name>
         </plugin>
     </gazebo>
